Commit message: Update ozymandias.urdf.xacro

File: ozymandias/urdf/ozymandias.urdf.xacro (robot description, xacro)
@@ -8,4 +8,8 @@
   <xacro:property name="radiusCylinder" value=".1" />
   <xacro:property name="lengthCylinder" value=".05" />
+  <!--post to elevate sensor properties-->
+  <xacro:property name="depthPost" value=".1" />
+  <xacro:property name="widthPost" value=".1" />
+  <xacro:property name="heightPost" value=".1" />
   <!--box body-->
   <link name="base_link">
@@ -14,8 +18,17 @@
         <box size="${depthBox} ${widthBox} ${heightBox}"/>
       </geometry>
-      <origin rpy="0 0 0" xyz="0 0 ${heightBox}"/>
+      <origin rpy="0 0 0" xyz="0 0 0"/>
     </visual>
   </link>
-  <!--algorithm for creating wheels and joints-->
+  <!--Post to elevate sensor-->
+  <link name="post">
+    <visual>
+      <geometry>
+        <box size="${depthPost} ${widthPost} ${heightPost}"/>
+      </geometry>
+      <origin rpy="0 0 0" xyz="0 0 0"/>
+    </visual>
+  </link>
+  <!--algorithm for creating wheels-->
   <xacro:macro name="wheel" params="prefix x y">
       <link name="${prefix}Wheel">
@@ -31,5 +44,5 @@
         <child link="${prefix}Wheel"/>
         <axis xyz="0 ${((widthBox/2)+(lengthCylinder/2))} 0"/>
-        <origin xyz="${((depthBox/2)-radiusCylinder)*x} ${((widthBox/2)+(lengthCylinder/2))*y} ${heightBox}"/>
+        <origin xyz="${((depthBox/2)-radiusCylinder)*x} ${((widthBox/2)+(lengthCylinder/2))*y} ${(heightBox/-2)}"/>
       </joint>
   </xacro:macro>
@@ -37,3 +50,15 @@
   <xacro:wheel prefix="rightFront" x="1" y="-1"/>
   <xacro:wheel prefix="leftFront" x="1" y="1"/>
+  <joint name="postToBodyJoint" type="fixed">
+    <parent link="base_link"/>
+    <child link="post"/>
+    <origin xyz="0 0 ${(heightBox/2)+(heightPost/2)}"/>
+  </joint>
+  <!-- need to make a placeholder link for the laser frame -->
+<link name="laser" />
+<joint name="laserToPost" type="fixed">
+    <parent link="post"/>
+    <child link="laser"/>
+    <origin rpy="0 0 3.1415" xyz="0 0 ${heightPost/2}"/>
+</joint>
 </robot>

Commit message: Update ozymandias.urdf.xacro

File: ozymandias/urdf/ozymandias.urdf.xacro (robot description, xacro)
@@ -2,14 +2,14 @@
 <robot xmlns:xacro="http://www.ros.org/wiki/xacro" name="ozymandias">
   <!--central box properties-->
-  <xacro:property name="depthBox" value=".5" />
-  <xacro:property name="widthBox" value=".3" />
-  <xacro:property name="heightBox" value=".1" />
+  <xacro:property name="depthBox" value="0.1778" />
+  <xacro:property name="widthBox" value="0.1778" />
+  <xacro:property name="heightBox" value="0.00635" />
   <!--wheel properties-->
-  <xacro:property name="radiusCylinder" value=".1" />
-  <xacro:property name="lengthCylinder" value=".05" />
+  <xacro:property name="radiusCylinder" value="0.032512" />
+  <xacro:property name="lengthCylinder" value="0.026162" />
   <!--post to elevate sensor properties-->
-  <xacro:property name="depthPost" value=".1" />
-  <xacro:property name="widthPost" value=".1" />
-  <xacro:property name="heightPost" value=".1" />
+  <xacro:property name="depthPost" value="0.127" />
+  <xacro:property name="widthPost" value="0.1016" />
+  <xacro:property name="heightPost" value="0.05715" />
   <!--box body-->
   <link name="base_link">
@@ -44,5 +44,5 @@
         <child link="${prefix}Wheel"/>
         <axis xyz="0 ${((widthBox/2)+(lengthCylinder/2))} 0"/>
-        <origin xyz="${((depthBox/2)-radiusCylinder)*x} ${((widthBox/2)+(lengthCylinder/2))*y} ${(heightBox/-2)}"/>
+        <origin xyz="${(depthBox/2)*x} ${((widthBox/2)+(lengthCylinder/2))*y} ${(heightBox/2)-radiusCylinder}"/>
       </joint>
   </xacro:macro>
@@ -53,5 +53,5 @@
     <parent link="base_link"/>
     <child link="post"/>
-    <origin xyz="0 0 ${(heightBox/2)+(heightPost/2)}"/>
+    <origin xyz="${depthPost/2+depthBox/2 - depthBox} 0 ${(heightBox/2)+(heightPost/2)}"/>
   </joint>
   <!-- need to make a placeholder link for the laser frame -->
@@ -60,5 +60,5 @@
     <parent link="post"/>
     <child link="laser"/>
-    <origin rpy="0 0 3.1415" xyz="0 0 ${heightPost/2}"/>
+    <origin rpy="0 0 3.1415" xyz="${depthPost/-4} 0 ${heightPost/2 + 0.0381}"/>
 </joint>
 </robot>
